File: ergogen/output/pcbs/scorn_choc_wireless.kicad_pcb (KiCad board)
At the start: 2 copper layers, 148.1 x 94.4 mm, 76 parts

Commit message: updated v1.1
Other:
- board text added: "v1.1_wl"
Changed lines of the file:
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@@
 		(at 197.866 147.32 180)
 		(property "Reference" "LOGO_B"
-			(at 0 0 360)
+			(at 0 0 0)
 			(layer "F.SilkS")
 			(hide yes)
@@
 		)
 		(property "Value" "LOGO"
-			(at 0.75 0 360)
+			(at 0.75 0 0)
 			(layer "F.SilkS")
 			(hide yes)
@@
 		)
 		(property "Footprint" "images:logo_sml"
-			(at 0 0 360)
+			(at 0 0 0)
 			(layer "F.Fab")
 			(hide yes)
@@
 		)
 		(property "Datasheet" ""
-			(at 0 0 360)
+			(at 0 0 0)
 			(layer "F.Fab")
 			(hide yes)
@@
 		)
 		(property "Description" ""
-			(at 0 0 360)
+			(at 0 0 0)
 			(layer "F.Fab")
 			(hide yes)
@@
 		)
 		(fp_line
-			(start 6.999997 6)
+			(start 6.999996 6)
 			(end 7 7)
 			(stroke
@@
 		(fp_line
 			(start 7 -7)
-			(end 6 -6.999997)
+			(end 6 -6.999996)
 			(stroke
 				(width 0.15)
@@
 		(fp_line
 			(start -7 7)
-			(end -6 6.999997)
+			(end -6 6.999996)
 			(stroke
 				(width 0.15)
@@
 		)
 		(fp_line
-			(start -6.999997 -6)
+			(start -6.999996 -6)
 			(end -7 -7)
 			(stroke
@@
 		)
 		(fp_line
-			(start 6.999997 6)
+			(start 6.999996 6)
 			(end 7 7)
 			(stroke
@@
 		(fp_line
 			(start 7 -7)
-			(end 6 -6.999997)
+			(end 6 -6.999996)
 			(stroke
 				(width 0.15)
@@
 		(fp_line
 			(start -7 7)
-			(end -6 6.999997)
+			(end -6 6.999996)
 			(stroke
 				(width 0.15)
@@
 		)
 		(fp_line
-			(start -6.999997 -6)
+			(start -6.999996 -6)
 			(end -7 -7)
 			(stroke
@@
 		)
 		(fp_line
-			(start 6.999997 6)
+			(start 6.999996 6)
 			(end 7 7)
 			(stroke
@@
 		(fp_line
 			(start 7 -7)
-			(end 6 -6.999997)
+			(end 6 -6.999996)
 			(stroke
 				(width 0.15)
@@
 		(fp_line
 			(start -7 7)
-			(end -6 6.999997)
+			(end -6 6.999996)
 			(stroke
 				(width 0.15)
@@
 		)
 		(fp_line
-			(start -6.999997 -6)
+			(start -6.999996 -6)
 			(end -7 -7)
 			(stroke
@@
 		(layer "Edge.Cuts")
 	)
+	(gr_text "v1.1_wl"
+		(at 271.526 167.132 65.5)
+		(layer "F.SilkS")
+		(effects
+			(font
+				(size 1 1)
+				(thickness 0.2)
+				(bold yes)
+			)
+			(justify left bottom)
+		)
+	)
 	(segment
